Commit message: make easier the tests

File: dummy_urdf.urdf (robot description, URDF)
Before this commit: robot JACO3_URDF_V11, 10 links, 9 joints
Links:
- link ForeArm_Link: mass 3.0 -> 1.0
- link HalfArm1_Link: mass 2.0 -> 1.0
- link HalfArm2_Link: mass 2.0 -> 1.0
- link Shoulder_Link: mass 2.0 -> 1.0
Joints:
- joint Actuator2: limit lower=-2.2 upper=2.2 effort=39 velocity=0.8727 -> lower=1.57 upper=2.2 effort=39 velocity=0.8727
- joint Actuator4: limit lower=-2.5656 upper=2.5656 effort=39 velocity=0.8727 -> lower=1.57 upper=2.5656 effort=39 velocity=0.8727
- joint Actuator6: limit lower=-2.05 upper=2.05 effort=9 velocity=0.8727 -> lower=1.57 upper=2.05 effort=9 velocity=0.8727

Commit message: Copied the paper test and realization of plots

File: dummy_urdf.urdf (robot description, URDF)
Before this commit: robot JACO3_URDF_V11, 10 links, 9 joints
Links:
- link Bracelet_Link: mass 1.0 -> 0.500657
- link ForeArm_Link: mass 1.0 -> 2.0
- link HalfArm1_Link: mass 1.0 -> 2.0
- link HalfArm2_Link: mass 1.0 -> 2.0
- link Shoulder_Link: mass 1.0 -> 2.0
- link SphericalWrist1_Link: mass 1.0 -> 2.0
- link SphericalWrist2_Link: mass 1.0 -> 2.0
Joints:
- joint Actuator2: limit lower=1.57 upper=2.2 effort=39 velocity=0.8727 -> lower=-2.2 upper=2.2 effort=39 velocity=0.8727
- joint Actuator4: limit lower=1.57 upper=2.5656 effort=39 velocity=0.8727 -> lower=-2.5656 upper=2.5656 effort=39 velocity=0.8727
- joint Actuator6: limit lower=1.57 upper=2.05 effort=9 velocity=0.8727 -> lower=-2.05 upper=2.05 effort=9 velocity=0.8727

Commit message: Testing everything

File: dummy_urdf.urdf (robot description, URDF)
Before this commit: robot JACO3_URDF_V11, 10 links, 9 joints
Links:
- link ForeArm_Link: mass 2.0 -> 0.930287
- link HalfArm1_Link: mass 2.0 -> 1.163667
- link HalfArm2_Link: mass 2.0 -> 1.16366
- link Shoulder_Link: mass 2.0 -> 1.377353
- link SphericalWrist1_Link: mass 2.0 -> 0.678106
- link SphericalWrist2_Link: mass 2.0 -> 0.678106
