Commit message: progressing know kinova shows

File: models/urdf/JACO3_URDF_V11.urdf (robot description, URDF)
Before this commit: robot JACO3_URDF_V11, 9 links, 8 joints
Links:
- added link world
- link Bracelet_Link: geometry collision mesh filename=../stl/Robot/Bracelet_Link.stl; visual mesh filename=../stl/Robot/Bracelet_Link.stl
- link ForeArm_Link: geometry collision mesh filename=../stl/Robot/ForeArm_Link.stl; visual mesh filename=../stl/Robot/ForeArm_Link.stl
- link HalfArm1_Link: geometry collision mesh filename=../stl/Robot/HalfArm1_Link.stl; visual mesh filename=../stl/Robot/HalfArm1_Link.stl
- link HalfArm2_Link: geometry collision mesh filename=../stl/Robot/HalfArm2_Link.stl; visual mesh filename=../stl/Robot/HalfArm2_Link.stl
- link Shoulder_Link: geometry collision mesh filename=../stl/Robot/Shoulder_Link.stl; visual mesh filename=../stl/Robot/Shoulder_Link.stl
- link SphericalWrist1_Link: geometry collision mesh filename=../stl/Robot/SphericalWrist1_Link.stl; visual mesh filename=../stl/Robot/SphericalWrist1_Link.stl
- link SphericalWrist2_Link: geometry collision mesh filename=../stl/Robot/SphericalWrist2_Link.stl; visual mesh filename=../stl/Robot/SphericalWrist2_Link.stl
- link base_link: geometry collision mesh filename=../stl/Robot/Base_Link.stl; visual mesh filename=../stl/Robot/Base_Link.stl
Joints:
- added joint world_joint: type fixed, parent world, child base_link, origin xyz=0.0 0.0 0.0 rpy=0.0 0.0 0

Commit message: modified to be able to modify the characteristics of a specific link or joint

File: models/urdf/JACO3_URDF_V11.urdf (robot description, URDF)
Before this commit: robot JACO3_URDF_V11, 10 links, 9 joints
Links:
- link EndEffector_Link: mass None -> 0.0

Commit message: New computation of the invers kinematics

File: models/urdf/JACO3_URDF_V11.urdf (robot description, URDF)
Before this commit: robot JACO3_URDF_V11, 10 links, 9 joints
Joints:
- joint world_joint: origin xyz=0.0 0.0 0.0 rpy=0.0 0.0 0 -> xyz=0.0 0.0 0.0 rpy=0.0 0.0 0.0
