Commit message: Last modifications

File: models/urdf/Cartesian_control.urdf (robot description, URDF)
Before this commit: robot Cartesian_control_URDF, 6 links, 5 joints
Joints:
- joint x_control_joint: limit lower=-3 upper=3 effort=1000.0 velocity=2 -> lower=-3 upper=3 effort=100.0 velocity=2
- joint y_control_joint: limit lower=-3 upper=3 effort=1000.0 velocity=2 -> lower=-3 upper=3 effort=100.0 velocity=2
- joint z_control_joint: limit lower=-3 upper=3 effort=1000.0 velocity=2 -> lower=-3 upper=3 effort=100.0 velocity=2
